Commit message: Registration part 1 implementation. Working on setting up connectivity to other parts of app

File: app/src/main/assets/V5_description/urdf/V5.urdf (robot description, URDF)
Before this commit: robot V5, 5 links, 4 joints
Links:
- added link tcp_link, mass 0.001; collision sphere radius=0.0005; visual sphere radius=0.0
Joints:
- added joint tcp_joint: type fixed, parent link_3_1, child tcp_link, origin xyz=-0.0065 0.082187 0.0254391 rpy=0 0 0

Commit message: Completed Registration Logic

File: app/src/main/assets/V5_description/urdf/V5.urdf (robot description, URDF)
Before this commit: robot V5, 6 links, 5 joints
Links:
- added link evd_link, mass 0.001; collision sphere radius=0.0; visual sphere radius=0.00
- link tcp_link: geometry collision sphere radius=0.0; visual sphere radius=0.00
Joints:
- added joint evd_joint: type fixed, parent link_3_1, child evd_link, origin xyz=-0.00175 0.079937 0.021542 rpy=0 0 0
- joint tcp_joint: origin xyz=-0.0065 0.082187 0.0254391 rpy=0 0 0 -> xyz=-0.00475 0.00225 0.0038971 rpy=0 0 0; parent link_3_1 -> evd_link
